File: ecad/afm.kicad_sch (KiCad schematic)
At the start: 1 part, among them J1 Conn_01x24

Commit message: apc stuff; rough block diagram
Parts:
- added JP1: Jumper_3_Open, Jumper:Jumper_Harwin_S1621_P10.9mm, symbol Jumper:Jumper_3_Open
Connections:
- net ACT_Focus+ renamed F+
- net ACT_Focus- renamed F-
- net ACT_Tracking+ renamed T+
- net T+: no longer J1.4 (Pin_4)
- net LD_DVD_LD renamed DVD_LD
- net LD_GND renamed GND_LD
- net LD_HFM_EN renamed HFM
- net LD_Monitor_Diode renamed MD
- net PDIC_CD_DVD_SW renamed CD_DVD_SW
- net PDIC_DVD_a renamed a
- net PDIC_DVD_b renamed b
- net PDIC_DVD_c renamed c
- net PDIC_DVD_d renamed d
- net PDIC_GND renamed GND_PD
- net PDIC_Vc renamed Vref
- net PDIC_Vcc renamed Vcc
- new net T-: J1.4 (Pin_4)
Other:
- added sheet ADCs (focus_signal_adc.kicad_sch)
- added sheet ADCs1 (focus_signal_adc.kicad_sch)
- added sheet Amplifier Stages (quadrant_amp_stages.kicad_sch)
- added sheet Amplifier Stages1 (quadrant_amp_stages.kicad_sch)
- added sheet MCU (mcu.kicad_sch)
- note added: "Actuator"
- note added: "Laser Diode"
- note added: "Photo detector"
- note added: "Piezo Driver stuff"
- note added: "SF-HD860 OPU"
- note added: "Voicecoil Driver stuff"
- note removed: "TODO: confirm which GNDs"

Commit message: bd; vca
Connections:
- net CD_DVD_SW is gone; now on net GND: J1.7 (Pin_7)
- net GND_LD is gone; now on net GND: J1.24 (Pin_24)
- net DVD_LD: now also JP1.2 (C)
- net GND: now also JP1.3 (B)
- net Laser APC/LD_DVD: now reaches JP1.1 (A)
- net F: now reaches J1.11 (Pin_11)
- net E: now reaches J1.15 (Pin_15)
- net VR_CD: now reaches J1.17 (Pin_17)
- net CD_LD: now reaches J1.19 (Pin_19)
- net PDIC_RF renamed RF
- net Vcc renamed +5V
- net Vref renamed +2V1
- no-connect marks 7 -> 8
Other:
- note added: "- [x] check if the PDIC and Laser have different GNDS: YES; can i still connect them? - [ ] schematic: unity-gain amps for FES buffers - [ ] figure out basic voicecoil driving. sch + proto - [ ] proto the LD apc. - [ ] characterize FES signals at focus levels (using voicecoils) - [ ] figure out if more signal conditioning is needed - [ ] research ADCs"
- note removed: "- [ ] check if the PDIC and Laser have different GNDS"
- moved on the sheet: JP1

Commit message: moar
Parts:
- removed J1: Conn_01x24, symbol Connector_Generic:Conn_01x24
- removed JP1: Jumper_3_Open, Jumper:Jumper_Harwin_S1621_P10.9mm, symbol Jumper:Jumper_3_Open
Connections:
- no-connect marks 8 -> 0
Other:
- removed sheet ADCs
- removed sheet ADCs1
- removed sheet Amplifier Stages
- removed sheet Amplifier Stages1
- added sheet OPU (opu.kicad_sch)
- added sheet PDIC Pre-processing (pdic_preproc.kicad_sch)
- note added: "- [x] check if the PDIC and Laser have different GNDS: YES; can i still connect them? - [x] schematic: unity-gain amps for FES buffers - [ ] figure out basic voicecoil driving. sch + proto - [ ] proto the LD apc. - [ ] characterize FES signals at focus levels (using voicecoils) - [ ] figure out if more signal conditioning is needed - [ ] research ADCs"
- note removed: "- [x] check if the PDIC and Laser have different GNDS: YES; can i still connect them? - [ ] schematic: unity-gain amps for FES buffers - [ ] figure out basic voicecoil driving. sch + proto - [ ] proto the LD apc. - [ ] characterize FES signals at focus levels (using voicecoils) - [ ] figure out if more signal conditioning is needed - [ ] research ADCs"
- note removed: "Actuator"
- note removed: "Laser Diode"
- note removed: "Photo detector"
- note removed: "SF-HD860 OPU"
