File: ecad/laser_apc.kicad_sch (KiCad schematic)
At the start: 14 parts, among them Q1 Q_PNP, U1 TL082

Commit message: apc stuff; rough block diagram
Parts:
- removed D2: ??, symbol Device:D
- removed U1: TL082, Package_DIP:DIP-8_W7.62mm, symbol Amplifier_Operational:TL082
- added D3: BAT54W, Package_TO_SOT_SMD:SOT-323_SC-70, symbol Diode:BAT54W
- added U2: MCP6002-xP, Package_DIP:DIP-8_W7.62mm, symbol Amplifier_Operational:MCP6002-xP
- Q1: value Q_PNP -> 2N2907A/MMBT2907A
Connections:
- net +5V: now also U2.8 (V+)
- net GND: now also D3.1 (A), U2.4 (V-)
- net LD_DVD: now also D3.3 (K)
- net MD: now also U2.3 (+)
- net VREF = 0.18V: now also U2.2 (-)
- net at R4.2, R5.1: now also U2.1
Other:
- moved on the sheet: C2

Commit message: moar
Connections:
- net GND renamed GND_LD
Changed lines of the file:
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@@
 			)
 		)
-		(property "Value" "GND"
-			(at 85.09 135.89 0)
+		(property "Value" "GND_LD"
+			(at 87.63 132.0799 0)
 			(show_name no)
 			(do_not_autoplace no)
@@
 					(size 1.27 1.27)
 				)
+				(justify left)
 			)
 		)
@@
 		)
 		(property "Value" "+5V"
-			(at 85.09 68.58 0)
+			(at 87.63 72.3899 0)
 			(show_name no)
 			(do_not_autoplace no)
@@
 					(size 1.27 1.27)
 				)
+				(justify left)
 			)
 		)

Commit message: things
Other:
- note added: "If too bright => MD current increases. (flows MD kathode to anode) => Raises voltage at Sense+ input. => Op-amp raises output voltage to help Sense- catch-up. => PNP bjt lowers current since base is closer to E => Lower LD brightness"
- note removed: "If too bright => reverse bias current produced. => Raises voltage at Sense+ input. => Op-amp raises output voltage to help Sense- catch-up. => PNP bjt lowers current if base closer to E => Lower LD brightness"
- title: (none) -> Laser Automatic Power Controller
Changed lines of the file:
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@@
 	(paper "A4")
 	(title_block
+		(title "Laser Automatic Power Controller")
+		(date "2026-07-17")
 		(rev "0.0.0")
 		(company "Hacker Fab")
 		(comment 1 "Yash Karthik")
+		(comment 4 "Verified: 2026-07-17")
 	)
 	(text "conn. to diode Anode (+)"
@@
 		)
 	)
-	(text "If too bright => reverse bias current produced.\n=> Raises voltage at Sense+ input.\n=> Op-amp raises output voltage to help Sense- catch-up.\n=> PNP bjt lowers current if base closer to E\n=> Lower LD brightness"
+	(text "If too bright => MD current increases. (flows MD kathode to anode)\n=> Raises voltage at Sense+ input.\n=> Op-amp raises output voltage to help Sense- catch-up.\n=> PNP bjt lowers current since base is closer to E\n=> Lower LD brightness"
 		(exclude_from_sim no)
 		(at 178.054 156.972 0)
