File: ecad/focus_signal_adc.kicad_sch (KiCad schematic)
At the start: 0 parts

Commit message: need to sweep
Other:
- note removed: "ADS1256?"
Changed lines of the file:
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@@
 		(comment 1 "Yash Karthik")
-	)
-	(text "ADS1256?"
-		(exclude_from_sim no)
-		(at 71.374 101.346 0)
-		(effects
-			(font
-				(size 1.27 1.27)
-			)
-		)
 	)
 	(hierarchical_label "Q2_digital"
