File: ecad/pdic_preproc.kicad_sch (KiCad schematic)
At the start: 0 parts

Commit message: need to sweep
Parts:
- added C14, C16, C7: 10nF, symbol Device:C_Small
- added R16, R18: 1K, symbol Device:R_US
- added U5: OPA2134, symbol Amplifier_Operational:OPA2134
Connections:
- net a_raw: now also R16.1
- net b_raw: now also R18.1
- new net: C14.1, R16.2, U5.3 (+)
- new net: C16.1, R18.2, U5.5 (+)
- new net +5V: C7.1, U5.8 (V+)
- new net GND: C14.2, C16.2
- new net GND_PD: C7.2, U5.4 (V-)
- new net Q1_amped: U5.1, U5.2 (-)
- new net Q2_amped: U5.6 (-), U5.7
Other:
- removed sheet ADCs
- removed sheet ADCs1
- removed sheet Amplifier Stages
- removed sheet Amplifier Stages1
- note added: "ADS1256?"
- note added: "TODO: check sec 6.2.3 Source Impedance and Distortion when ADC finalized"
