File: ecad/quadrant_amp_stages.kicad_sch (KiCad schematic)
At the start: 1 part, among them U1 OPA2134

Commit message: moar
Parts:
- added C6: 10nF, symbol Device:C_Small
- renumbered U1 to U4
Connections:
- net Q1_amped: now also U4.1, U4.2 (-)
- net Q1_raw: now also U4.3 (+)
- net Q2_amped: now also U4.6 (-), U4.7
- net Q2_raw: now also U4.5 (+)
- net GND_PD: now reaches U4.4 (V-)
- net GND_PD: now also C6.2
- net +5V: now reaches U4.8 (V+)
- net +5V: now also C6.1
Other:
- note added: "TODO: check sec 6.2.3 Source Impedance and Distortion when ADC finalized"
- note added: "filter?"
- title: (none) -> PDIC Amplifier Stages
- moved on the sheet: U4A, U4B, U4C

Commit message: vca sims
Parts:
- added C13, C15: 10nF, symbol Device:C_Small
- added R15, R17: 1K, symbol Device:R_US
Connections:
- net Q1_raw: now also R15.1; no longer U4.3 (+)
- net Q2_raw: now also R17.1; no longer U4.5 (+)
- new net: C13.1, R15.2, U4.3 (+)
- new net: C15.1, R17.2, U4.5 (+)
- new net GND: C13.2, C15.2
Other:
- note removed: "filter?"

Commit message: need to sweep
Parts:
- removed C13, C15, C6: 10nF, symbol Device:C_Small
- removed R15, R17: 1K, symbol Device:R_US
- removed U4: OPA2134, symbol Amplifier_Operational:OPA2134
Other:
- note removed: "TODO: check sec 6.2.3 Source Impedance and Distortion when ADC finalized"
