File: ecad/vca_driver.kicad_sch (KiCad schematic)
At the start: 21 parts, among them Q2 BD140, Q4 BD139, Q5 BD139, U3 OPA2277

Commit message: change val
Parts:
- R12: value 2R -> 3.3K
- R20: value 2R -> 3K
Changed lines of the file:
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@@
 		(lib_id "Device:R_US")
 		(at 152.4 96.52 0)
-		(mirror y)
-		(unit 1)
-		(body_style 1)
-		(exclude_from_sim no)
-		(in_bom yes)
-		(on_board yes)
-		(in_pos_files yes)
-		(dnp no)
-		(fields_autoplaced yes)
+		(unit 1)
+		(body_style 1)
+		(exclude_from_sim no)
+		(in_bom yes)
+		(on_board yes)
+		(in_pos_files yes)
+		(dnp no)
 		(property "Reference" "R20"
 			(at 149.86 95.2499 0)
@@
 					(size 1.27 1.27)
 				)
-				(justify left)
-			)
-		)
-		(property "Value" "2R"
+				(justify right)
+			)
+		)
+		(property "Value" "3K"
 			(at 149.86 97.7899 0)
 			(show_name no)
@@
 					(size 1.27 1.27)
 				)
-				(justify left)
+				(justify right)
 			)
 		)
 		(property "Footprint" ""
-			(at 151.384 96.774 90)
+			(at 153.416 96.774 90)
 			(hide yes)
 			(show_name no)
@@
 			)
 		)
-		(property "Value" "2R"
+		(property "Value" "3.3K"
 			(at 151.13 85.09 0)
 			(show_name no)

Commit message: reorg; dac symbols
Parts:
- removed unit 2 of U3
Connections:
- no-connect marks 3 -> 0
Other:
- note added: "U3's part B in MCU/DAC page."
Changed lines of the file:
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@@
+		)
+	)
+	(text "U3's part B in MCU/DAC page."
+		(exclude_from_sim no)
+		(at 160.274 195.072 0)
+		(effects
+			(font
+				(size 1.27 1.27)
+			)
 		)
 	)
@@
 		(diameter 0)
 		(color 0 0 0 0)
-	)
-	(no_connect
-		(at 266.7 31.75)
-	)
-	(no_connect
-		(at 266.7 26.67)
-	)
-	(no_connect
-		(at 281.94 29.21)
 	)
 	(wire
@@
 				)
 			)
-		)
-	)
-	(symbol
-		(lib_id "Amplifier_Operational:OPA2277")
-		(at 274.32 29.21 0)
-		(unit 2)
-		(body_style 1)
-		(exclude_from_sim no)
-		(in_bom yes)
-		(on_board yes)
-		(in_pos_files yes)
-		(dnp no)
-		(fields_autoplaced yes)
-		(property "Reference" "U3"
-			(at 274.32 19.05 0)
-			(show_name no)
-			(do_not_autoplace no)
-			(effects
-				(font
-					(size 1.27 1.27)
-				)
-			)
-		)
-		(property "Value" "OPA2277"
-			(at 274.32 21.59 0)
-			(show_name no)
-			(do_not_autoplace no)
-			(effects
-				(font
-					(size 1.27 1.27)
-				)
-			)
-		)
-		(property "Footprint" ""
-			(at 274.32 29.21 0)
-			(hide yes)
-			(show_name no)
-			(do_not_autoplace no)
-			(effects
-				(font
-					(size 1.27 1.27)
-				)
-			)
-		)
-		(property "Datasheet" "https://www.ti.com/lit/ds/symlink/opa2277.pdf"
-			(at 274.32 29.21 0)
-			(hide yes)
-			(show_name no)
-			(do_not_autoplace no)
-			(effects
-				(font
-					(size 1.27 1.27)
-				)
-			)
-		)
-		(property "Description" "Dual High Precision Operational Amplifiers, DIP-8/SOIC-8"
-			(at 274.32 29.21 0)
-			(hide yes)
-			(show_name no)
-			(do_not_autoplace no)
-			(effects
-				(font
-					(size 1.27 1.27)
-				)
-			)
-		)
-		(pin "8"
-		)
-		(pin "4"
-		)
-		(pin "6"
-		)
-		(pin "5"
-		)
-		(pin "7"
-		)
-		(pin "3"
-		)
-		(pin "1"
-		)
-		(pin "2"
-		)
-		(instances
-			(project "afm"
-				(path "/62de9aa8-4539-4ecb-8acc-2c7a46b3005b/152e488a-5c59-4955-a770-fd5dc463781b"
-					(reference "U3")
-					(unit 2)
-				)
-			)

Commit message: vca drv ref
Parts:
- added R25, R27: 10K, symbol Device:R_US
- added R26, R28: 1.6K, symbol Device:R_US
- added unit 2 of U3
Connections:
- net DRV_CURR_Vref: now also R27.1
- net GND: now also R28.2
- net at R14.1, U3.3 (+): now also R26.2, U3.7
- new net: R25.2, R26.1, U3.6 (-)
- new net: R27.2, R28.1, U3.5 (+)
- new net DAC_MIDPT: R25.1
Other:
- note added: "Level Shift + Fractional Gain Stage"
- note added: "Vout = 0.16*DRV - 0.2V scales 0-2.5V to 0-0.4V shifts -200mV => -200mV to 200mV range"
- note removed: "Some sort of clamp to limit max Vref to ~0.3V"
- note removed: "U3's part B in MCU/DAC page."
- note removed: "level-shifter stage"
- moved on the sheet: C10, C11, C12, C5, C9, D2, D4, Q2, Q4, Q5, R10, R11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

Commit message: need to sweep
Connections:
- net DAC_MIDPT renamed DAC_MIDPT_Vref
- net DRV_CURR_Vref renamed VCA_DRV
Changed lines of the file:
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@@
 		)
 	)
-	(hierarchical_label "DAC_MIDPT"
+	(hierarchical_label "DAC_MIDPT_Vref"
 		(shape input)
 		(at 40.64 86.36 180)
@@
 		)
 	)
-	(hierarchical_label "DRV_CURR_Vref"
+	(hierarchical_label "VCA_DRV"
 		(shape input)
 		(at 40.64 91.44 180)
